File: KiCAD/SignalStrengthRecorder/SignalStrengthRecorder.sch (KiCad schematic (older format))
At the start: 11 parts, among them U1 ADC0831-2CH, U2 ADC0831-2CH, U3 ADC0831-2CH, U4 ADC0831-2CH, U5 ADC0831-2CH

Commit message: work in progress
Parts:
- removed J?: Conn_02x20_Odd_Even, symbol Connector_Generic:Conn_02x20_Odd_Even
- added J?: Radio1, symbol Connector:Conn_01x03_Male
- added J?: Raspberry_Pi_2_3, symbol Connector:Raspberry_Pi_2_3
- added J?: Radio2, symbol Connector:Conn_01x03_Male
- added J?: Radio3, symbol Connector:Conn_01x03_Male
- added J?: Radio4, symbol Connector:Conn_01x03_Male
- added J?: Radio5, symbol Connector:Conn_01x03_Male
- added R? (x5): R, symbol Device:R
- K?: symbol SignalStrengthRecorder:HFE8 -> SignalStrengthRecorder-rescue:HFE8-SignalStrengthRecorder
- U1, U2, U3, U4, U5: symbol SignalStrengthRecorder:ADC0831-2CH -> SignalStrengthRecorder-rescue:ADC0831-2CH-SignalStrengthRecorder
Connections:
- net labels added: Radio1Active, Radio2Active, Radio3Active, Radio4Active, Radio5Active
- wire segments 86 -> 128
Other:
- moved on the sheet: Q?, R?

Commit message: annotated diag04 diagram, added datasheet for PN2222 NPN transistor, modified schematic.  ***Need to check latching relay circuit and pinouts***
Parts:
- removed Q? (x2): Q_NPN_ECB, symbol Device:Q_NPN_ECB
- added Q? (x2): Q_NPN_EBC, symbol Device:Q_NPN_EBC
Connections:
- wire segments 128 -> 134
- no-connect marks 0 -> 2
Changed lines of the file:
@@
 	1    0    0    -1
-$EndComp
-$Comp
-L Device:Q_NPN_ECB Q?
-U 1 1 5BEA9CF5
-P 9945 5220
-F 0 "Q?" H 10135 5174 50  0000 L CNN
-F 1 "Q_NPN_ECB" H 10135 5265 50  0000 L CNN
-F 2 "" H 10145 5320 50  0001 C CNN
-F 3 "~" H 9945 5220 50  0001 C CNN
-	1    9945 5220
-	-1   0    0    1
-$EndComp
-$Comp
-L Device:Q_NPN_ECB Q?
-U 1 1 5BEA9E34
-P 9325 5935
-F 0 "Q?" H 9515 5889 50  0000 L CNN
-F 1 "Q_NPN_ECB" H 9515 5980 50  0000 L CNN
-F 2 "" H 9525 6035 50  0001 C CNN
-F 3 "~" H 9325 5935 50  0001 C CNN
-	1    9325 5935
-	-1   0    0    1
 $EndComp
 Text GLabel 8825 3920 1    50   Input ~ 0
 +5V
-Text GLabel 8925 3920 1    50   Input ~ 0
-+5V
 Wire Wire Line
 	8825 3920 8825 3990
-Wire Wire Line
-	8925 3920 8925 3990
 Text GLabel 8825 4890 3    50   Input ~ 0
 Vcc
@@
 Wire Wire Line
 	10440 2320 10300 2320
+Text GLabel 8570 1620 0    50   Input ~ 0
+CLK
+Wire Wire Line
+	8700 1620 8570 1620
+Text GLabel 8570 1520 0    50   Input ~ 0
+CS
+Wire Wire Line
+	8700 1520 8570 1520
+Text GLabel 10440 1420 2    50   Input ~ 0
+DO2
+Wire Wire Line
+	10300 1420 10440 1420
+Text GLabel 10440 1520 2    50   Input ~ 0
+DO3
+Wire Wire Line
+	10440 1520 10300 1520
+Text GLabel 10440 1720 2    50   Input ~ 0
+DO4
+Wire Wire Line
+	10440 1720 10300 1720
+Text GLabel 10440 1820 2    50   Input ~ 0
+DO5
+Wire Wire Line
+	10440 1820 10300 1820
+Text GLabel 8570 2620 0    50   Input ~ 0
+DO1
+Wire Wire Line
+	8700 2620 8570 2620
+$Comp
+L Device:Q_NPN_EBC Q?
+U 1 1 5C3B763A
+P 9945 5220
+F 0 "Q?" H 10135 5266 50  0000 L CNN
+F 1 "Q_NPN_EBC" H 10135 5175 50  0000 L CNN
+F 2 "" H 10145 5320 50  0001 C CNN
+F 3 "~" H 9945 5220 50  0001 C CNN
+	1    9945 5220
+	-1   0    0    -1
+$EndComp
+$Comp
+L Device:Q_NPN_EBC Q?
+U 1 1 5C3BCCD4
+P 9325 5935
+F 0 "Q?" H 9515 5981 50  0000 L CNN
+F 1 "Q_NPN_EBC" H 9515 5890 50  0000 L CNN
+F 2 "" H 9525 6035 50  0001 C CNN
+F 3 "~" H 9325 5935 50  0001 C CNN
+	1    9325 5935
+	-1   0    0    -1
+$EndComp
+NoConn ~ 8925 4790
+NoConn ~ 8925 3985
 $EndSCHEMATC

Commit message: modified schematic to power the latching coil from Rpi's pin 2, 5V
Connections:
- net labels added: Rpi_5V
- wire segments 134 -> 136
Changed lines of the file:
@@
 	9845 5420 9845 5490
 Text GLabel 9225 3920 1    50   Input ~ 0
-+5V
+Rpi_5V
 Text GLabel 9325 3920 1    50   Input ~ 0
-+5V
+Rpi_5V
 Wire Wire Line
 	9225 3920 9225 3990
@@
 NoConn ~ 8925 4790
 NoConn ~ 8925 3985
+Text GLabel 9150 685  0    50   Input ~ 0
+Rpi_5V
+Wire Wire Line
+	9150 685  9300 685
+Wire Wire Line
+	9300 685  9300 720
 $EndSCHEMATC
